File: hardware/stm32f1DevBoard.sch (KiCad schematic (older format))
At the start: 15 parts

Commit message: more schematic
Parts:
- removed C? (x4): 0.1uF, symbol CSMALL
- added C?: 0.1uF, symbol CSMALL
- added JP?: BOOT0, symbol JUMPER_3X1
- added R?: 10k, symbol R
- added U1: STM32F102C6, symbol STM32F102C6
- gave numbers to parts that had none: 11
Connections:
- wire segments 38 -> 49
Other:
- moved on the sheet: S1, X1, X2

Commit message: power
Parts:
- added BT1: BATTERY, symbol BATTERY
- added C1, C3: 10uF, symbol CSMALL
- added C2: 100uF, symbol CSMALL
- added C4: 1uF, symbol CSMALL
- added D1: DIODE, symbol DIODE
- added J1: POWER_JACK, symbol POWER_JACK
- added J2: USB_2, symbol USB_2
- added JP1: JUMPER_3X1, symbol JUMPER_3X1
- added JP3: JTAG_ENABLE, symbol JUMPER_2X1
- added P1: JTAG, symbol JTAG
- added Q1: MOSFET-N, symbol MOSFET-N
- added R1, R2, R3, R4: ?, symbol R
- added R10, R11, R9: 10k, symbol R
- added R5: 1k5, symbol R
- added R7, R8: 22, symbol R
- added U2: LM358, symbol LM358
- added U?: VREG_GNDCENTER, symbol VREG_GNDCENTER
- added U?: VREG_VOUTCENTER, symbol VREG_VOUTCENTER
- gave numbers to parts that had none: 3
- renumbered C6 to C11, C7 to C12, C8 to C13, C1 to C5, C2 to C6, C3 to C7, C4 to C8, C5 to C9, U1 to U4
Connections:
- net labels added: +5V, JTCK, JTDI, JTDO, JTMS, VBAT, VIN, VUSB, nJTRST, nRST
- wire segments 49 -> 154
- no-connect marks 0 -> 26
Other:
- moved on the sheet: S1

Commit message: wifi and sdcard
Parts:
- removed C2: 100uF, symbol CSMALL
- added C11: 100uF, symbol CPSMALL
- added C14: 10uF, symbol CSMALL
- added C15, C16, C?: 0.1uF, symbol CSMALL
- added D?: POWER, symbol LED
- added J?: SDCARD, symbol SDCARD
- added JP?: WIFIRESET, symbol JUMPER_2X1
- added JP?: WIFIWP, symbol JUMPER_2X1
- added JP?: WIFIHIBERNATE, symbol JUMPER_2X1
- added JP?: WIFIINT, symbol JUMPER_2X1
- added JP?: WIFICS, symbol JUMPER_2X1
- added P?: WIFIDEBUG, symbol P03
- added P? (x2): P20, symbol P20
- added R10, R11, R12, R13, R9, R?: 10k, symbol R
- added R?: ?, symbol R
- added U5: MRF24WB0MX, symbol MRF24WB0MX
- gave numbers to parts that had none: 2
- renumbered C4 to C1, C13 to C10, C3 to C12, C1 to C13, C5 to C2, C6 to C3, C7 to C4, C8 to C5, C9 to C6, C10 to C7, C11 to C8, C12 to C9, J2 to J1, J1 to J2, JP2 to JP1, JP1 to JP2, R9 to R14, R10 to R15, R11 to R16, U2 to U1
Connections:
- net labels added: MISO, MOSI, RX1, RX2, SCK, SDCS, TX1, TX2, WIFIHIBERNATE, nWIFICS, nWIFIINT, nWIFIRESET, nWIFIWP
- wire segments 154 -> 275
- no-connect marks 26 -> 0
Other:
- moved on the sheet: BT1, J1, JP1, JP2, JP3, P1, R14, R15, R16, R5, R6, R7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

Commit message: seperate into sheets
Parts:
- removed BT1: BATTERY, symbol BATTERY
- removed C11: 100uF, symbol CPSMALL
- removed C12, C13, C14: 10uF, symbol CSMALL
- removed C15, C16, C?: 0.1uF, symbol CSMALL
- removed D1: DIODE, symbol DIODE
- removed D?: POWER, symbol LED
- removed J2: POWER_JACK, symbol POWER_JACK
- removed J?: SDCARD, symbol SDCARD
- removed JP2: JUMPER_3X1, symbol JUMPER_3X1
- removed JP?: WIFIRESET, symbol JUMPER_2X1
- removed JP?: WIFIWP, symbol JUMPER_2X1
- removed JP?: WIFIHIBERNATE, symbol JUMPER_2X1
- removed JP?: WIFIINT, symbol JUMPER_2X1
- removed JP?: WIFICS, symbol JUMPER_2X1
- removed P?: WIFIDEBUG, symbol P03
- removed Q1: MOSFET-N, symbol MOSFET-N
- removed R1, R2, R3, R4, R?: ?, symbol R
- removed R10, R11, R12, R13, R9: 10k, symbol R
- removed U1: LM358, symbol LM358
- removed U2: VREG_GNDCENTER, symbol VREG_GNDCENTER
- removed U3: VREG_VOUTCENTER, symbol VREG_VOUTCENTER
- removed U5: MRF24WB0MX, symbol MRF24WB0MX
- gave numbers to parts that had none: 3
- renumbered JP3 to JP1, JP1 to JP2, R14 to R1, R15 to R2, R16 to R3, R5 to R4, R6 to R5, R7 to R6, R8 to R7, U4 to U1
Connections:
- net labels removed: VIN
- wire segments 275 -> 146
- no-connect marks 0 -> 3
Other:
- moved on the sheet: J1, JP1, JP2, P1, P2, P3, R1, R2, R3, R4, R5, R6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

Commit message: pcb initial layout
Parts:
- added M1, M2, M3, M4: Mounting Hole, symbol MECH
- C3, C4, C8, C9: value 0.1uF -> 22pF
Changed lines of the file:
@@
-EESchema Schematic File Version 2  date Sun 16 Dec 2012 11:20:27 PM EST
+EESchema Schematic File Version 2  date Tue 18 Dec 2012 10:27:06 PM EST
 LIBS:stm32f1DevBoard
 LIBS:power
@@
 Sheet 1 4
 Title ""
-Date "17 dec 2012"
+Date "19 dec 2012"
 Rev ""
 Comp ""
@@
 F 1 "32,768Hz" H 3550 2275 60  0000 C CNN
 	1    3550 2400
-	1    0    0    -1
+	-1   0    0    1
 $EndComp
 $Comp
@@
 P 3800 2550
 F 0 "C8" H 3825 2600 30  0000 L CNN
-F 1 "0.1uF" H 3825 2500 30  0000 L CNN
+F 1 "22pF" H 3825 2500 30  0000 L CNN
 	1    3800 2550
 	1    0    0    -1
@@
 P 3300 2550
 F 0 "C3" H 3325 2600 30  0000 L CNN
-F 1 "0.1uF" H 3325 2500 30  0000 L CNN
+F 1 "22pF" H 3325 2500 30  0000 L CNN
 	1    3300 2550
 	1    0    0    -1
@@
 P 3800 3050
 F 0 "C9" H 3825 3100 30  0000 L CNN
-F 1 "0.1uF" H 3825 3000 30  0000 L CNN
+F 1 "22pF" H 3825 3000 30  0000 L CNN
 	1    3800 3050
 	1    0    0    -1
@@
 P 3300 3050
 F 0 "C4" H 3325 3100 30  0000 L CNN
-F 1 "0.1uF" H 3325 3000 30  0000 L CNN
+F 1 "22pF" H 3325 3000 30  0000 L CNN
 	1    3300 3050
 	1    0    0    -1
@@
 Wire Wire Line
 	4350 1950 4400 1950
+$Comp
+L MECH M1
+U 1 1 50D1344C
+P 5700 5800
+F 0 "M1" H 5750 5800 60  0000 C CNN
+F 1 "Mounting Hole" H 5900 5800 60  0000 L CNN
+	1    5700 5800
+	1    0    0    -1
+$EndComp
+$Comp
+L MECH M2
+U 1 1 50D13459
+P 5700 5900
+F 0 "M2" H 5750 5900 60  0000 C CNN
+F 1 "Mounting Hole" H 5900 5900 60  0000 L CNN
+	1    5700 5900
+	1    0    0    -1
+$EndComp
+$Comp
+L MECH M3
+U 1 1 50D1345F
+P 5700 6000
+F 0 "M3" H 5750 6000 60  0000 C CNN
+F 1 "Mounting Hole" H 5900 6000 60  0000 L CNN
+	1    5700 6000
+	1    0    0    -1
+$EndComp
+$Comp
+L MECH M4
+U 1 1 50D13465
+P 5700 6100
+F 0 "M4" H 5750 6100 60  0000 C CNN
+F 1 "Mounting Hole" H 5900 6100 60  0000 L CNN
+	1    5700 6100
+	1    0    0    -1
+$EndComp
 $EndSCHEMATC

Commit message: switched transistor
Parts:
- added F1: FUSE, symbol FUSE
Connections:
- wire segments 146 -> 147
Other:
- moved on the sheet: J1
Changed lines of the file:
@@
-EESchema Schematic File Version 2  date Tue 18 Dec 2012 10:27:06 PM EST
+EESchema Schematic File Version 2  date Wed 19 Dec 2012 08:51:07 PM EST
 LIBS:stm32f1DevBoard
 LIBS:power
@@
 $EndDescr
 $Comp
-L +3.3V #PWR01
+L +3.3V #PWR18
 U 1 1 50C949CA
 P 4300 1450
-F 0 "#PWR01" H 4300 1410 30  0001 C CNN
+F 0 "#PWR18" H 4300 1410 30  0001 C CNN
 F 1 "+3.3V" H 4300 1560 30  0000 C CNN
 	1    4300 1450
@@
 $EndComp
 $Comp
-L GND #PWR02
+L GND #PWR10
 U 1 1 50C94D41
 P 3300 2050
-F 0 "#PWR02" H 3300 2050 30  0001 C CNN
+F 0 "#PWR10" H 3300 2050 30  0001 C CNN
 F 1 "GND" H 3300 1980 30  0001 C CNN
 	1    3300 2050
@@
 $EndComp
 $Comp
-L GND #PWR03
+L GND #PWR6
 U 1 1 50C9550D
 P 3000 4250
-F 0 "#PWR03" H 3000 4250 30  0001 C CNN
+F 0 "#PWR6" H 3000 4250 30  0001 C CNN
 F 1 "GND" H 3000 4180 30  0001 C CNN
 	1    3000 4250
@@
 $EndComp
 $Comp
-L GND #PWR04
+L GND #PWR19
 U 1 1 50C95BDE
 P 4300 4850
-F 0 "#PWR04" H 4300 4850 30  0001 C CNN
+F 0 "#PWR19" H 4300 4850 30  0001 C CNN
 F 1 "GND" H 4300 4780 30  0001 C CNN
 	1    4300 4850
@@
 $EndComp
 $Comp
-L GND #PWR05
+L GND #PWR11
 U 1 1 50CA07BA
 P 3300 2700
-F 0 "#PWR05" H 3300 2700 30  0001 C CNN
+F 0 "#PWR11" H 3300 2700 30  0001 C CNN
 F 1 "GND" H 3300 2630 30  0001 C CNN
 	1    3300 2700
@@
 $EndComp
 $Comp
-L GND #PWR06
+L GND #PWR14
 U 1 1 50CA07C0
 P 3800 2700
-F 0 "#PWR06" H 3800 2700 30  0001 C CNN
+F 0 "#PWR14" H 3800 2700 30  0001 C CNN
 F 1 "GND" H 3800 2630 30  0001 C CNN
 	1    3800 2700
@@
 $EndComp
 $Comp
-L GND #PWR07
+L GND #PWR12
 U 1 1 50CA07C6
 P 3300 3200
-F 0 "#PWR07" H 3300 3200 30  0001 C CNN
+F 0 "#PWR12" H 3300 3200 30  0001 C CNN
 F 1 "GND" H 3300 3130 30  0001 C CNN
 	1    3300 3200
@@
 $EndComp
 $Comp
-L GND #PWR08
+L GND #PWR15
 U 1 1 50CA07CC
 P 3800 3200
-F 0 "#PWR08" H 3800 3200 30  0001 C CNN
+F 0 "#PWR15" H 3800 3200 30  0001 C CNN
 F 1 "GND" H 3800 3130 30  0001 C CNN
 	1    3800 3200
@@
 $EndComp
 $Comp
-L GND #PWR09
+L GND #PWR13
 U 1 1 50CA0DC0
 P 3750 4450
-F 0 "#PWR09" H 3750 4450 30  0001 C CNN
+F 0 "#PWR13" H 3750 4450 30  0001 C CNN
 F 1 "GND" H 3750 4380 30  0001 C CNN
 	1    3750 4450
@@
 $EndComp
 $Comp
-L GND #PWR010
+L GND #PWR8
 U 1 1 50C9FD3B
 P 3000 5000
-F 0 "#PWR010" H 3000 5000 30  0001 C CNN
+F 0 "#PWR8" H 3000 5000 30  0001 C CNN
 F 1 "GND" H 3000 4930 30  0001 C CNN
 	1    3000 5000
@@
 $EndComp
 $Comp
-L +3.3V #PWR011
+L +3.3V #PWR7
 U 1 1 50C9FD41
 P 3000 4700
-F 0 "#PWR011" H 3000 4660 30  0001 C CNN
+F 0 "#PWR7" H 3000 4660 30  0001 C CNN
 F 1 "+3.3V" H 3000 4810 30  0000 C CNN
 	1    3000 4700
@@
 $EndComp
 $Comp
-L GND #PWR012
+L GND #PWR17
 U 1 1 50CBE59B
 P 3900 6950
-F 0 "#PWR012" H 3900 6950 30  0001 C CNN
+F 0 "#PWR17" H 3900 6950 30  0001 C CNN
 F 1 "GND" H 3900 6880 30  0001 C CNN
 	1    3900 6950
@@
 $EndComp
 $Comp
-L +3.3V #PWR013
+L +3.3V #PWR16
 U 1 1 50CBE85F
 P 3900 5850
-F 0 "#PWR013" H 3900 5810 30  0001 C CNN
+F 0 "#PWR16" H 3900 5810 30  0001 C CNN
 F 1 "+3.3V" H 3900 5960 30  0000 C CNN
 	1    3900 5850
@@
 $EndComp
 $Comp
-L +3.3V #PWR014
+L +3.3V #PWR3
 U 1 1 50CBE8C7
 P 2400 5850
-F 0 "#PWR014" H 2400 5810 30  0001 C CNN
+F 0 "#PWR3" H 2400 5810 30  0001 C CNN
 F 1 "+3.3V" H 2400 5960 30  0000 C CNN
 	1    2400 5850
@@
 $EndComp
 $Comp
-L GND #PWR015
+L GND #PWR4
 U 1 1 50CBE96B
 P 2400 7400
-F 0 "#PWR015" H 2400 7400 30  0001 C CNN
+F 0 "#PWR4" H 2400 7400 30  0001 C CNN
 F 1 "GND" H 2400 7330 30  0001 C CNN
 	1    2400 7400
@@
 $EndComp
 $Comp
-L GND #PWR016
+L GND #PWR2
 U 1 1 50CBE971
 P 2100 7400
-F 0 "#PWR016" H 2100 7400 30  0001 C CNN
+F 0 "#PWR2" H 2100 7400 30  0001 C CNN
 F 1 "GND" H 2100 7330 30  0001 C CNN
 	1    2100 7400
@@
 $EndComp
 $Comp
-L GND #PWR017
+L GND #PWR1
 U 1 1 50CBE977
 P 1800 7400
-F 0 "#PWR017" H 1800 7400 30  0001 C CNN
+F 0 "#PWR1" H 1800 7400 30  0001 C CNN
 F 1 "GND" H 1800 7330 30  0001 C CNN
 	1    1800 7400
@@
 L USB_2 J1
 U 1 1 50CC0796
-P 2400 3500
-F 0 "J1" H 2325 3750 60  0000 C CNN
-F 1 "USB_2" H 2450 3200 60  0001 C CNN
-F 4 "VCC" H 2725 3650 50  0001 C CNN "VCC"
-F 5 "D+" H 2700 3550 50  0001 C CNN "Data+"
-F 6 "D-" H 2700 3450 50  0001 C CNN "Data-"
-F 7 "GND" H 2725 3350 50  0001 C CNN "Ground"
-	1    2400 3500
+P 1600 3500
+F 0 "J1" H 1525 3750 60  0000 C CNN
+F 1 "USB_2" H 1650 3200 60  0001 C CNN
+F 4 "VCC" H 1925 3650 50  0001 C CNN "VCC"
+F 5 "D+" H 1900 3550 50  0001 C CNN "Data+"
+F 6 "D-" H 1900 3450 50  0001 C CNN "Data-"
+F 7 "GND" H 1925 3350 50  0001 C CNN "Ground"
+	1    1600 3500
 	1    0    0    -1
 $EndComp
@@
 $EndComp
 $Comp
-L GND #PWR018
+L GND #PWR5
 U 1 1 50CC0E79
 P 2700 3750
-F 0 "#PWR018" H 2700 3750 30  0001 C CNN
+F 0 "#PWR5" H 2700 3750 30  0001 C CNN
 F 1 "GND" H 2700 3680 30  0001 C CNN
 	1    2700 3750
@@
 $EndComp
 $Comp
-L +3.3V #PWR019
+L +3.3V #PWR9
 U 1 1 50CC1031
 P 3050 2950
-F 0 "#PWR019" H 3050 2910 30  0001 C CNN
+F 0 "#PWR9" H 3050 2910 30  0001 C CNN
 F 1 "+3.3V" H 3050 3060 30  0000 C CNN
 	1    3050 2950
@@
 	3850 3350 3850 3450
 Wire Wire Line
-	3850 3450 2600 3450
+	3850 3450 1800 3450
 Wire Wire Line
 	3900 3650 3850 3650
@@
 	3850 3650 3850 3550
 Wire Wire Line
-	3850 3550 2600 3550
-Wire Wire Line
-	2600 3650 2700 3650
+	3850 3550 1800 3550
+Wire Wire Line
+	1800 3650 2700 3650
 Wire Wire Line
 	2700 3650 2700 3750
@@
 	7300 4650 8350 4650
 $Comp
-L GND #PWR020
+L GND #PWR26
 U 1 1 50CD9603
 P 9100 3550
-F 0 "#PWR020" H 9100 3550 30  0001 C CNN
+F 0 "#PWR26" H 9100 3550 30  0001 C CNN
 F 1 "GND" H 9100 3480 30  0001 C CNN
 	1    9100 3550
@@
 $EndComp
 $Comp
-L GND #PWR021
+L GND #PWR23
 U 1 1 50CD9609
 P 8250 5050
-F 0 "#PWR021" H 8250 5050 30  0001 C CNN
+F 0 "#PWR23" H 8250 5050 30  0001 C CNN
 F 1 "GND" H 8250 4980 30  0001 C CNN
 	1    8250 5050
@@
 	9100 3450 9100 3550
 $Comp
-L +3.3V #PWR022
+L +3.3V #PWR25
 U 1 1 50CD9878
 P 9100 1450
-F 0 "#PWR022" H 9100 1410 30  0001 C CNN
+F 0 "#PWR25" H 9100 1410 30  0001 C CNN
 F 1 "+3.3V" H 9100 1560 30  0000 C CNN
 	1    9100 1450
@@
 $EndComp
 $Comp
-L +3.3V #PWR023
+L +3.3V #PWR22
 U 1 1 50CD987E
 P 8250 1450
-F 0 "#PWR023" H 8250 1410 30  0001 C CNN
+F 0 "#PWR22" H 8250 1410 30  0001 C CNN
 F 1 "+3.3V" H 8250 1560 30  0000 C CNN
 	1    8250 1450
@@
 	9100 3350 9100 1450
 $Comp
-L +5V #PWR024
+L +5V #PWR21
 U 1 1 50CD9B00
 P 8150 1450
-F 0 "#PWR024" H 8150 1540 20  0001 C CNN
+F 0 "#PWR21" H 8150 1540 20  0001 C CNN
 F 1 "+5V" H 8150 1540 30  0000 C CNN
 	1    8150 1450
@@
 $EndComp
 $Comp
-L GND #PWR025
+L GND #PWR20
 U 1 1 50CDC19E
 P 7950 5250
-F 0 "#PWR025" H 7950 5250 30  0001 C CNN
+F 0 "#PWR20" H 7950 5250 30  0001 C CNN
 F 1 "GND" H 7950 5180 30  0001 C CNN
 	1    7950 5250
@@
 JTDI
 $Comp
-L +5V #PWR026
+L +5V #PWR24
 U 1 1 50CE57F4
 P 9000 1450
-F 0 "#PWR026" H 9000 1540 20  0001 C CNN
+F 0 "#PWR24" H 9000 1540 20  0001 C CNN
 F 1 "+5V" H 9000 1540 30  0000 C CNN
 	1    9000 1450
@@
 NoConn ~ 9200 3050
 NoConn ~ 9200 3150
-Wire Wire Line
-	2600 3350 2650 3350
 Wire Wire Line
 	4350 1950 4400 1950
@@
 	1    0    0    -1
 $EndComp
+$Comp
+L FUSE F1
+U 1 1 50D1CB86
+P 2200 3350
+F 0 "F1" H 2300 3400 40  0000 C CNN
+F 1 "FUSE" H 2100 3300 40  0000 C CNN
+	1    2200 3350
+	1    0    0    -1
+$EndComp
+Wire Wire Line
+	1800 3350 1950 3350
+Wire Wire Line
+	2450 3350 2650 3350
 $EndSCHEMATC
