File: hardware/stm32f1DevBoard-WiFi.sch (KiCad schematic (older format))
At the start: 15 parts, among them P4 WIFIDEBUG, U2 MRF24WB0MX

Commit message: using kicadcloud files
Parts:
- C11, C12, C13: symbol CSMALL -> CPsmall
Changed lines of the file:
@@
-EESchema Schematic File Version 2  date Wed 19 Dec 2012 11:05:56 PM EST
-LIBS:stm32f1DevBoard
+EESchema Schematic File Version 2  date Wed 02 Jan 2013 12:15:05 PM EST
+LIBS:userFavorites
 LIBS:power
-LIBS:device
-LIBS:transistors
-LIBS:conn
-LIBS:linear
-LIBS:regul
-LIBS:74xx
-LIBS:cmos4000
-LIBS:adc-dac
-LIBS:memory
-LIBS:xilinx
-LIBS:special
-LIBS:microcontrollers
-LIBS:dsp
-LIBS:microchip
-LIBS:analog_switches
-LIBS:motorola
-LIBS:texas
-LIBS:intel
-LIBS:audio
-LIBS:interface
-LIBS:digital-audio
-LIBS:philips
-LIBS:display
-LIBS:cypress
-LIBS:siliconi
-LIBS:opto
-LIBS:atmel
-LIBS:contrib
-LIBS:valves
-LIBS:stm32f1DevBoard-cache
 EELAYER 27 0
 EELAYER END
@@
 $EndComp
 $Comp
-L CSMALL C11
+L CPsmall C11
 U 1 1 50CE2658
 P 5900 2200
@@
 $EndComp
 $Comp
-L CSMALL C12
+L CPsmall C12
 U 1 1 50CE265E
 P 6100 2200
@@
 $EndComp
 $Comp
-L CSMALL C13
+L CPsmall C13
 U 1 1 50CE2664
 P 6300 2200
