File: hardware/stm32f1DevBoard-power.sch (KiCad schematic (older format))
At the start: 17 parts, among them J2 POWER_JACK, Q1 MOSFET-P, U3 LM358, U4 VREG-X-5, U5 VREG-5-3.3

Commit message: update hardware
Parts:
- removed D1: DIODE, symbol DIODE
- added C18: 100uF, symbol CPSMALL
- added D1: DIODESCH, symbol DIODESCH
Connections:
- wire segments 62 -> 63
Other:
- note added: "Pin2 = 2.5V\nPin3 = 2.5V at 7.65V"
- moved on the sheet: C16
Changed lines of the file:
@@
-EESchema Schematic File Version 2  date Thu 31 Jan 2013 11:01:55 PM EST
+EESchema Schematic File Version 2  date Tue 12 Feb 2013 08:34:35 PM EST
 LIBS:userFavorites
 LIBS:power
@@
 Sheet 3 4
 Title ""
-Date "1 feb 2013"
+Date "13 feb 2013"
 Rev ""
 Comp ""
@@
 $EndComp
 $Comp
-L GND #PWR038
+L GND #PWR041
 U 1 1 50CE2BF2
 P 2100 1800
-F 0 "#PWR038" H 2100 1800 30  0001 C CNN
+F 0 "#PWR041" H 2100 1800 30  0001 C CNN
 F 1 "GND" H 2100 1730 30  0001 C CNN
 	1    2100 1800
@@
 $EndComp
 $Comp
-L +3.3V #PWR039
+L +3.3V #PWR042
 U 1 1 50CE2BF8
 P 2900 1300
-F 0 "#PWR039" H 2900 1260 30  0001 C CNN
+F 0 "#PWR042" H 2900 1260 30  0001 C CNN
 F 1 "+3.3V" H 2900 1410 30  0000 C CNN
 	1    2900 1300
@@
 $EndComp
 $Comp
-L DIODE D1
-U 1 1 50CE2C0B
-P 2800 3650
-F 0 "D1" H 2800 3750 40  0000 C CNN
-F 1 "DIODE" H 2800 3550 40  0000 C CNN
-	1    2800 3650
-	1    0    0    -1
-$EndComp
-$Comp
-L GND #PWR040
+L GND #PWR043
 U 1 1 50CE2C12
 P 2600 3950
-F 0 "#PWR040" H 2600 3950 30  0001 C CNN
+F 0 "#PWR043" H 2600 3950 30  0001 C CNN
 F 1 "GND" H 2600 3880 30  0001 C CNN
 	1    2600 3950
@@
 $EndComp
 $Comp
-L GND #PWR041
+L GND #PWR044
 U 1 1 50CE2C18
 P 3600 4050
-F 0 "#PWR041" H 3600 4050 30  0001 C CNN
+F 0 "#PWR044" H 3600 4050 30  0001 C CNN
 F 1 "GND" H 3600 3980 30  0001 C CNN
 	1    3600 4050
@@
 $EndComp
 $Comp
-L +5V #PWR042
+L +5V #PWR045
 U 1 1 50CE2C1E
 P 4500 3550
-F 0 "#PWR042" H 4500 3640 20  0001 C CNN
+F 0 "#PWR045" H 4500 3640 20  0001 C CNN
 F 1 "+5V" H 4500 3640 30  0000 C CNN
 	1    4500 3550
@@
 $EndComp
 $Comp
-L GND #PWR043
+L GND #PWR046
 U 1 1 50CE2C2A
 P 4200 4050
-F 0 "#PWR043" H 4200 4050 30  0001 C CNN
+F 0 "#PWR046" H 4200 4050 30  0001 C CNN
 F 1 "GND" H 4200 3980 30  0001 C CNN
 	1    4200 4050
@@
 $EndComp
 $Comp
-L +5V #PWR044
+L +5V #PWR047
 U 1 1 50CE2C4E
 P 2700 5550
-F 0 "#PWR044" H 2700 5640 20  0001 C CNN
+F 0 "#PWR047" H 2700 5640 20  0001 C CNN
 F 1 "+5V" H 2700 5640 30  0000 C CNN
 	1    2700 5550
@@
 $EndComp
 $Comp
-L GND #PWR045
+L GND #PWR048
 U 1 1 50CE2C55
 P 2400 6800
-F 0 "#PWR045" H 2400 6800 30  0001 C CNN
+F 0 "#PWR048" H 2400 6800 30  0001 C CNN
 F 1 "GND" H 2400 6730 30  0001 C CNN
 	1    2400 6800
@@
 $EndComp
 $Comp
-L GND #PWR046
+L GND #PWR049
 U 1 1 50CE2C5B
 P 3200 6600
-F 0 "#PWR046" H 3200 6600 30  0001 C CNN
+F 0 "#PWR049" H 3200 6600 30  0001 C CNN
 F 1 "GND" H 3200 6530 30  0001 C CNN
 	1    3200 6600
@@
 $EndComp
 $Comp
-L +5V #PWR047
+L +5V #PWR050
 U 1 1 50CE2C61
 P 3200 5700
-F 0 "#PWR047" H 3200 5790 20  0001 C CNN
+F 0 "#PWR050" H 3200 5790 20  0001 C CNN
 F 1 "+5V" H 3200 5790 30  0000 C CNN
 	1    3200 5700
@@
 $EndComp
 $Comp
-L +5V #PWR048
+L +5V #PWR051
 U 1 1 50CE2C6E
 P 5900 6250
-F 0 "#PWR048" H 5900 6340 20  0001 C CNN
+F 0 "#PWR051" H 5900 6340 20  0001 C CNN
 F 1 "+5V" H 5900 6340 30  0000 C CNN
 	1    5900 6250
@@
 $EndComp
 $Comp
-L GND #PWR049
+L GND #PWR052
 U 1 1 50CE2C74
 P 8150 4100
-F 0 "#PWR049" H 8150 4100 30  0001 C CNN
+F 0 "#PWR052" H 8150 4100 30  0001 C CNN
 F 1 "GND" H 8150 4030 30  0001 C CNN
 	1    8150 4100
@@
 $EndComp
 $Comp
-L +3.3V #PWR050
+L +3.3V #PWR053
 U 1 1 50CE2C7A
-P 8850 3650
-F 0 "#PWR050" H 8850 3610 30  0001 C CNN
-F 1 "+3.3V" H 8850 3760 30  0000 C CNN
-	1    8850 3650
+P 9000 3650
+F 0 "#PWR053" H 9000 3610 30  0001 C CNN
+F 1 "+3.3V" H 9000 3760 30  0000 C CNN
+	1    9000 3650
 	1    0    0    -1
 $EndComp
@@
 L CPsmall C16
 U 1 1 50CE2C80
-P 8750 4050
-F 0 "C16" H 8775 4100 30  0000 L CNN
-F 1 "10uF" H 8775 4000 30  0000 L CNN
-	1    8750 4050
-	1    0    0    -1
-$EndComp
-$Comp
-L GND #PWR051
+P 9000 4000
+F 0 "C16" H 9025 4050 30  0000 L CNN
+F 1 "10uF" H 9025 3950 30  0000 L CNN
+	1    9000 4000
+	1    0    0    -1
+$EndComp
+$Comp
+L GND #PWR054
 U 1 1 50CE2C86
-P 8750 4200
-F 0 "#PWR051" H 8750 4200 30  0001 C CNN
-F 1 "GND" H 8750 4130 30  0001 C CNN
-	1    8750 4200
-	1    0    0    -1
-$EndComp
-$Comp
-L +5V #PWR052
+P 9000 4200
+F 0 "#PWR054" H 9000 4200 30  0001 C CNN
+F 1 "GND" H 9000 4130 30  0001 C CNN
+	1    9000 4200
+	1    0    0    -1
+$EndComp
+$Comp
+L +5V #PWR055
 U 1 1 50CE2C8C
 P 7650 3600
-F 0 "#PWR052" H 7650 3690 20  0001 C CNN
+F 0 "#PWR055" H 7650 3690 20  0001 C CNN
 F 1 "+5V" H 7650 3690 30  0000 C CNN
 	1    7650 3600
@@
 	5900 6550 5600 6550
 Wire Wire Line
-	8550 3750 8850 3750
+	8550 3750 9000 3750
 Wire Wire Line
 	8600 3750 8600 3850
 Wire Wire Line
 	8600 3850 8550 3850
-Wire Wire Line
-	8850 3750 8850 3650
 Connection ~ 8600 3750
 Wire Wire Line
-	8750 3750 8750 3950
-Connection ~ 8750 3750
-Wire Wire Line
-	8750 4150 8750 4200
+	9000 4100 9000 4200
 Wire Wire Line
 	7750 3750 7650 3750
@@
 $EndComp
 $Comp
-L GND #PWR053
+L GND #PWR056
 U 1 1 50CE2CF6
 P 8850 1700
-F 0 "#PWR053" H 8850 1700 30  0001 C CNN
+F 0 "#PWR056" H 8850 1700 30  0001 C CNN
 F 1 "GND" H 8850 1630 30  0001 C CNN
 	1    8850 1700
@@
 	8350 1600 8200 1600
 $Comp
-L +3.3V #PWR054
+L +3.3V #PWR057
 U 1 1 50CE2CFF
 P 7750 1500
-F 0 "#PWR054" H 7750 1460 30  0001 C CNN
+F 0 "#PWR057" H 7750 1460 30  0001 C CNN
 F 1 "+3.3V" H 7750 1610 30  0000 C CNN
 	1    7750 1500
@@
 Connection ~ 5100 6250
 $Comp
-L GND #PWR055
+L GND #PWR058
 U 1 1 50CEA124
 P 4400 6700
-F 0 "#PWR055" H 4400 6700 30  0001 C CNN
+F 0 "#PWR058" H 4400 6700 30  0001 C CNN
 F 1 "GND" H 4400 6630 30  0001 C CNN
 	1    4400 6700
@@
 $EndComp
 $Comp
-L +5V #PWR056
+L +5V #PWR059
 U 1 1 50CEA12A
 P 4400 5800
-F 0 "#PWR056" H 4400 5890 20  0001 C CNN
+F 0 "#PWR059" H 4400 5890 20  0001 C CNN
 F 1 "+5V" H 4400 5890 30  0000 C CNN
 	1    4400 5800
@@
 	1    0    0    -1
 $EndComp
+$Comp
+L CPSMALL C18
+U 1 1 510BDE91
+P 8750 4000
+F 0 "C18" H 8775 4050 30  0000 L CNN
+F 1 "100uF" H 8775 3950 30  0000 L CNN
+	1    8750 4000
+	1    0    0    -1
+$EndComp
+Wire Wire Line
+	9000 3650 9000 3900
+Connection ~ 9000 3750
+Wire Wire Line
+	8750 3750 8750 3900
+Connection ~ 8750 3750
+$Comp
+L GND #PWR060
+U 1 1 510BDF83
+P 8750 4200
+F 0 "#PWR060" H 8750 4200 30  0001 C CNN
+F 1 "GND" H 8750 4130 30  0001 C CNN
+	1    8750 4200
+	1    0    0    -1
+$EndComp
+Wire Wire Line
+	8750 4100 8750 4200
+Text Notes 2950 5350 0    60   ~ 0
+Pin2 = 2.5V\nPin3 = 2.5V at 7.65V
+$Comp
+L DIODESCH D1
+U 1 1 511AEE72
+P 2800 3650
+F 0 "D1" H 2800 3750 40  0000 C CNN
+F 1 "DIODESCH" H 2800 3550 40  0000 C CNN
+	1    2800 3650
+	1    0    0    -1
+$EndComp
